File: hardware/preamp/preamp.sch (KiCad schematic (older format))
At the start: 30 parts, among them J1 I/O, J2 Conn 2, J4 Conn 1, Q1 2SC3324, Q2 2SC3324, U1 TLV170DBV

Commit message: Updated PCB
Parts:
- renumbered J4 to J2, J2 to J3, R8 to R1, R1 to R10, R2 to R11, R3 to R12, R4 to R13, R5 to R14, R6 to R15, R7 to R16, R9 to R2, R10 to R3, R11 to R4, R12 to R5, R13 to R6, R14 to R7, R15 to R8, R16 to R9
Changed lines of the file:
@@
 $EndComp
 $Comp
-L power:GND #PWR0101
+L power:GND #PWR03
 U 1 1 60CA6062
 P 2200 4400
-F 0 "#PWR0101" H 2200 4150 50  0001 C CNN
+F 0 "#PWR03" H 2200 4150 50  0001 C CNN
 F 1 "GND" H 2205 4227 50  0000 C CNN
 F 2 "" H 2200 4400 50  0001 C CNN
@@
 $EndComp
 $Comp
-L power:GND #PWR0102
+L power:GND #PWR011
 U 1 1 60CBE4A7
 P 8100 3600
-F 0 "#PWR0102" H 8100 3350 50  0001 C CNN
+F 0 "#PWR011" H 8100 3350 50  0001 C CNN
 F 1 "GND" H 8105 3427 50  0000 C CNN
 F 2 "" H 8100 3600 50  0001 C CNN
@@
 $EndComp
 $Comp
-L power:GND #PWR0103
+L power:GND #PWR010
 U 1 1 60CC59EA
 P 7900 4800
-F 0 "#PWR0103" H 7900 4550 50  0001 C CNN
+F 0 "#PWR010" H 7900 4550 50  0001 C CNN
 F 1 "GND" H 7905 4627 50  0000 C CNN
 F 2 "" H 7900 4800 50  0001 C CNN
@@
 $EndComp
 $Comp
-L Device:R R6
+L Device:R R15
 U 1 1 60CE0F70
 P 9400 4900
-F 0 "R6" H 9470 4946 50  0000 L CNN
+F 0 "R15" H 9470 4946 50  0000 L CNN
 F 1 "10k" H 9470 4855 50  0000 L CNN
 F 2 "Resistor_SMD:R_0402_1005Metric" V 9330 4900 50  0001 C CNN
@@
 $EndComp
 $Comp
-L Device:R R7
+L Device:R R16
 U 1 1 60CE1D3D
 P 9800 4500
-F 0 "R7" V 9593 4500 50  0000 C CNN
+F 0 "R16" V 9593 4500 50  0000 C CNN
 F 1 "4.7k" V 9684 4500 50  0000 C CNN
 F 2 "Resistor_SMD:R_0402_1005Metric" V 9730 4500 50  0001 C CNN
@@
 mix
 $Comp
-L power:GND #PWR0108
+L power:GND #PWR012
 U 1 1 60CE2F96
 P 9400 5200
-F 0 "#PWR0108" H 9400 4950 50  0001 C CNN
+F 0 "#PWR012" H 9400 4950 50  0001 C CNN
 F 1 "GND" H 9405 5027 50  0000 C CNN
 F 2 "" H 9400 5200 50  0001 C CNN
@@
 $EndComp
 $Comp
-L power:GND #PWR0109
+L power:GND #PWR02
 U 1 1 60D40697
 P 2200 3600
-F 0 "#PWR0109" H 2200 3350 50  0001 C CNN
+F 0 "#PWR02" H 2200 3350 50  0001 C CNN
 F 1 "GND" H 2205 3427 50  0000 C CNN
 F 2 "" H 2200 3600 50  0001 C CNN
@@
 $EndComp
 $Comp
-L Device:R R1
+L Device:R R10
 U 1 1 60CA74D0
 P 6550 4400
-F 0 "R1" V 6343 4400 50  0000 C CNN
+F 0 "R10" V 6343 4400 50  0000 C CNN
 F 1 "39k" V 6434 4400 50  0000 C CNN
 F 2 "Resistor_SMD:R_0402_1005Metric" V 6480 4400 50  0001 C CNN
@@
 $EndComp
 $Comp
-L Device:R R2
+L Device:R R11
 U 1 1 60CA8735
 P 6550 4600
-F 0 "R2" V 6343 4600 50  0000 C CNN
+F 0 "R11" V 6343 4600 50  0000 C CNN
 F 1 "39k" V 6434 4600 50  0000 C CNN
 F 2 "Resistor_SMD:R_0402_1005Metric" V 6480 4600 50  0001 C CNN
@@
 $EndComp
 $Comp
-L Device:R R5
+L Device:R R14
 U 1 1 60CAA986
 P 8000 5250
-F 0 "R5" V 7900 5250 50  0000 C CNN
+F 0 "R14" V 7900 5250 50  0000 C CNN
 F 1 "91k" V 7800 5250 50  0000 C CNN
 F 2 "Resistor_SMD:R_0402_1005Metric" V 7930 5250 50  0001 C CNN
@@
 $EndComp
 $Comp
-L Device:R R3
+L Device:R R12
 U 1 1 60CA90D5
 P 7100 3500
-F 0 "R3" V 7307 3500 50  0000 C CNN
+F 0 "R12" V 7307 3500 50  0000 C CNN
 F 1 "180k" V 7216 3500 50  0000 C CNN
 F 2 "Resistor_SMD:R_0402_1005Metric" V 7030 3500 50  0001 C CNN
@@
 $EndComp
 $Comp
-L Device:R R4
+L Device:R R13
 U 1 1 60CAA1E5
 P 7700 3500
-F 0 "R4" V 7907 3500 50  0000 C CNN
+F 0 "R13" V 7907 3500 50  0000 C CNN
 F 1 "180k" V 7816 3500 50  0000 C CNN
 F 2 "Resistor_SMD:R_0402_1005Metric" V 7630 3500 50  0001 C CNN
@@
 Main Coil
 $Comp
-L power:PWR_FLAG #FLG0101
+L power:PWR_FLAG #FLG02
 U 1 1 60D54A12
 P 6400 1300
-F 0 "#FLG0101" H 6400 1375 50  0001 C CNN
+F 0 "#FLG02" H 6400 1375 50  0001 C CNN
 F 1 "PWR_FLAG" H 6400 1450 50  0000 C CNN
 F 2 "" H 6400 1300 50  0001 C CNN
@@
 V+
 $Comp
-L power:GND #PWR0105
+L power:GND #PWR07
 U 1 1 60CCD190
 P 5750 2000
-F 0 "#PWR0105" H 5750 1750 50  0001 C CNN
+F 0 "#PWR07" H 5750 1750 50  0001 C CNN
 F 1 "GND" H 5755 1827 50  0000 C CNN
 F 2 "" H 5750 2000 50  0001 C CNN
@@
 $EndComp
 $Comp
-L power:GND #PWR0104
+L power:GND #PWR09
 U 1 1 60CCC3D1
 P 6400 2000
-F 0 "#PWR0104" H 6400 1750 50  0001 C CNN
+F 0 "#PWR09" H 6400 1750 50  0001 C CNN
 F 1 "GND" H 6405 1827 50  0000 C CNN
 F 2 "" H 6400 2000 50  0001 C CNN
@@
 5, 4, 3: External coil\n2, 1: External coil shunt
 $Comp
-L power:GND #PWR0107
+L power:GND #PWR01
 U 1 1 60CC841D
 P 1800 2000
-F 0 "#PWR0107" H 1800 1750 50  0001 C CNN
+F 0 "#PWR01" H 1800 1750 50  0001 C CNN
 F 1 "GND" H 1800 1800 50  0000 C CNN
 F 2 "" H 1800 2000 50  0001 C CNN
@@
 ext_coil+
 $Comp
-L Connector_Generic:Conn_02x03_Counter_Clockwise J4
+L Connector_Generic:Conn_02x03_Counter_Clockwise J2
 U 1 1 60CA3D47
 P 2600 3600
-F 0 "J4" H 2650 3400 50  0000 C CNN
+F 0 "J2" H 2650 3400 50  0000 C CNN
 F 1 "Conn 1" H 2650 3850 50  0000 C CNN
 F 2 "cycfi_library:pin_socket_2x3p_1.00mm_smd_vertical" H 2600 3600 50  0001 C CNN
@@
 $EndComp
 $Comp
-L power:PWR_FLAG #FLG02
+L power:PWR_FLAG #FLG01
 U 1 1 60D52BC1
 P 3500 2000
-F 0 "#FLG02" H 3500 2075 50  0001 C CNN
+F 0 "#FLG01" H 3500 2075 50  0001 C CNN
 F 1 "PWR_FLAG" H 3350 2200 50  0000 C CNN
 F 2 "" H 3500 2000 50  0001 C CNN
@@
 $EndComp
 $Comp
-L power:GND #PWR0106
+L power:GND #PWR04
 U 1 1 60CDB5FB
 P 3300 2000
-F 0 "#PWR0106" H 3300 1750 50  0001 C CNN
+F 0 "#PWR04" H 3300 1750 50  0001 C CNN
 F 1 "GND" H 3300 1800 50  0000 C CNN
 F 2 "" H 3300 2000 50  0001 C CNN
@@
 $EndComp
 $Comp
-L Connector_Generic:Conn_02x03_Counter_Clockwise J2
+L Connector_Generic:Conn_02x03_Counter_Clockwise J3
 U 1 1 610F68E1
 P 2600 4400
-F 0 "J2" H 2650 4200 50  0000 C CNN
+F 0 "J3" H 2650 4200 50  0000 C CNN
 F 1 "Conn 2" H 2650 4650 50  0000 C CNN
 F 2 "cycfi_library:pin_socket_2x3p_1.00mm_smd_vertical" H 2600 4400 50  0001 C CNN
@@
 $EndComp
 $Comp
-L Device:R R10
+L Device:R R3
 U 1 1 611411EA
 P 4500 4100
-F 0 "R10" V 4293 4100 50  0000 C CNN
+F 0 "R3" V 4293 4100 50  0000 C CNN
 F 1 "39k" V 4384 4100 50  0000 C CNN
 F 2 "Resistor_SMD:R_0402_1005Metric" V 4430 4100 50  0001 C CNN
@@
 $EndComp
 $Comp
-L Device:R R13
+L Device:R R6
 U 1 1 61141C48
 P 5350 4100
-F 0 "R13" V 5143 4100 50  0000 C CNN
+F 0 "R6" V 5143 4100 50  0000 C CNN
 F 1 "39k" V 5234 4100 50  0000 C CNN
 F 2 "Resistor_SMD:R_0402_1005Metric" V 5280 4100 50  0001 C CNN
@@
 $EndComp
 $Comp
-L Device:R R8
+L Device:R R1
 U 1 1 61143602
 P 4100 4100
-F 0 "R8" V 3893 4100 50  0000 C CNN
+F 0 "R1" V 3893 4100 50  0000 C CNN
 F 1 "100k" V 3984 4100 50  0000 C CNN
 F 2 "Resistor_SMD:R_0402_1005Metric" V 4030 4100 50  0001 C CNN
@@
 $EndComp
 $Comp
-L Device:R R15
+L Device:R R8
 U 1 1 6114410D
 P 5750 4100
-F 0 "R15" V 5543 4100 50  0000 C CNN
+F 0 "R8" V 5543 4100 50  0000 C CNN
 F 1 "100k" V 5634 4100 50  0000 C CNN
 F 2 "Resistor_SMD:R_0402_1005Metric" V 5680 4100 50  0001 C CNN
@@
 $EndComp
 $Comp
-L Device:R R9
+L Device:R R2
 U 1 1 61144934
 P 4100 5450
-F 0 "R9" V 3893 5450 50  0000 C CNN
+F 0 "R2" V 3893 5450 50  0000 C CNN
 F 1 "51k" V 3984 5450 50  0000 C CNN
 F 2 "Resistor_SMD:R_0402_1005Metric" V 4030 5450 50  0001 C CNN
@@
 $EndComp
 $Comp
-L Device:R R16
+L Device:R R9
 U 1 1 61144F4B
 P 5750 5450
-F 0 "R16" V 5543 5450 50  0000 C CNN
+F 0 "R9" V 5543 5450 50  0000 C CNN
 F 1 "51k" V 5634 5450 50  0000 C CNN
 F 2 "Resistor_SMD:R_0402_1005Metric" V 5680 5450 50  0001 C CNN
@@
 $EndComp
 $Comp
-L Device:R R11
+L Device:R R4
 U 1 1 6114546E
 P 4500 5450
-F 0 "R11" V 4293 5450 50  0000 C CNN
+F 0 "R4" V 4293 5450 50  0000 C CNN
 F 1 "1.5k" V 4384 5450 50  0000 C CNN
 F 2 "Resistor_SMD:R_0402_1005Metric" V 4430 5450 50  0001 C CNN
@@
 $EndComp
 $Comp
-L Device:R R14
+L Device:R R7
 U 1 1 61145C43
 P 5350 5450
-F 0 "R14" V 5143 5450 50  0000 C CNN
+F 0 "R7" V 5143 5450 50  0000 C CNN
 F 1 "1.5k" V 5234 5450 50  0000 C CNN
 F 2 "Resistor_SMD:R_0402_1005Metric" V 5280 5450 50  0001 C CNN
@@
 $EndComp
 $Comp
-L Device:R R12
+L Device:R R5
 U 1 1 61145F48
 P 4950 5950
-F 0 "R12" V 4743 5950 50  0000 C CNN
+F 0 "R5" V 4743 5950 50  0000 C CNN
 F 1 "1.5k" V 4834 5950 50  0000 C CNN
 F 2 "Resistor_SMD:R_0402_1005Metric" V 4880 5950 50  0001 C CNN
@@
 $EndComp
 $Comp
-L power:GND #PWR0110
+L power:GND #PWR06
 U 1 1 6114655A
 P 4950 6350
-F 0 "#PWR0110" H 4950 6100 50  0001 C CNN
+F 0 "#PWR06" H 4950 6100 50  0001 C CNN
 F 1 "GND" H 4955 6177 50  0000 C CNN
 F 2 "" H 4950 6350 50  0001 C CNN
@@
 $EndComp
 $Comp
-L power:GND #PWR0111
+L power:GND #PWR05
 U 1 1 61146961
 P 4100 5800
-F 0 "#PWR0111" H 4100 5550 50  0001 C CNN
+F 0 "#PWR05" H 4100 5550 50  0001 C CNN
 F 1 "GND" H 4105 5627 50  0000 C CNN
 F 2 "" H 4100 5800 50  0001 C CNN
@@
 $EndComp
 $Comp
-L power:GND #PWR0112
+L power:GND #PWR08
 U 1 1 61146D18
 P 5750 5800
-F 0 "#PWR0112" H 5750 5550 50  0001 C CNN
+F 0 "#PWR08" H 5750 5550 50  0001 C CNN
 F 1 "GND" H 5755 5627 50  0000 C CNN
 F 2 "" H 5750 5800 50  0001 C CNN

Commit message: Added coil jumper
Parts:
- added JP1: Coil Shunt, Jumper:SolderJumper-2_P1.3mm_Open_TrianglePad1.0x1.5mm, symbol Jumper:Jumper_2_Open
Connections:
- net ext_coil-: now also JP1.1 (A)
- net in-: now also JP1.2 (B)
Changed lines of the file:
@@
 U 1 1 60CA2D4C
 P 8000 4500
-F 0 "U1" H 8100 4300 50  0000 L CNN
+F 0 "U1" H 8100 4300 50  0001 L CNN
 F 1 "TLV170DBV" H 8100 4200 50  0000 L CNN
 F 2 "Package_TO_SOT_SMD:SOT-23-5" H 7900 4300 50  0001 L CNN
@@
 Wire Wire Line
 	5300 1450 5150 1450
+$Comp
+L Jumper:Jumper_2_Open JP1
+U 1 1 61378A1B
+P 3050 3950
+F 0 "JP1" V 3004 4048 50  0000 L CNN
+F 1 "Coil Shunt" V 3095 4048 50  0000 L CNN
+F 2 "Jumper:SolderJumper-2_P1.3mm_Open_TrianglePad1.0x1.5mm" H 3050 3950 50  0001 C CNN
+F 3 "~" H 3050 3950 50  0001 C CNN
+	1    3050 3950
+	0    1    1    0
+$EndComp
+Wire Wire Line
+	3050 3750 3050 3600
+Connection ~ 3050 3600
+Wire Wire Line
+	3050 4150 2900 4150
+Wire Wire Line
+	2900 4150 2900 4300
+Connection ~ 2900 4300
 $EndSCHEMATC
