File: hardware/bobbin-bottom-3.3/bobbin-bottom-3.3/bobbin-bottom-3.3.kicad_pcb (KiCad board)
At the start: 2 copper layers, 68 x 8 mm, 5 parts

Commit message: Updated bobbin-bottom
Parts:
- removed IC, OC: MountingHole_Pad, cycfi_library:single-pad-3x3-th
- removed Out: Conn_01x03, cycfi_library:pad_1x03_P2.54mm
- H3: footprint cycfi_library:single-pad-3x1.5 -> cycfi_library:round-single-pad-1.8mm-th
- H4: footprint bobbin-bottom-3.3:core-pad -> cycfi_library:single-pad-10x2
- moved H3 74.0 mm to (98.3, 104.9)
- moved H4 43.1 mm to (130.0, 98.4)
Routing:
- net /OC: track 48.9 -> 0.00 mm
- net /IC: track 17.8 -> 0.00 mm
- net GND: track 36.8 -> 37.8 mm, vias 4 -> 0
Other:
- board size 68 x 8 mm -> 68.5 x 8.5 mm
