File: hardware/passive/passive.kicad_sch (KiCad schematic)
At the start: 7 parts, among them J1 i/O, J2 Conn 1, J3 Conn 2

Commit message: v2.0 layout
Parts:
- removed J2: Conn 1, cycfi_library:pin_socket_2x3p_1.00mm_smd_vertical, symbol Connector_Generic:Conn_02x03_Counter_Clockwise
- removed J3: Conn 2, cycfi_library:pin_socket_2x3p_1.00mm_smd_vertical, symbol Connector_Generic:Conn_02x03_Counter_Clockwise
- added J2: conn_2x2, cycfi_library:pin_socket_2x2p_2.00mm_smd_vertical, symbol Connector_Generic:Conn_02x02_Counter_Clockwise
- J1: value i/O -> I/O
Connections:
- net GND: now also J2.2 (Pin_2)
- net int_coil+: now also J2.4 (Pin_4)
- net out-: now also J2.3 (Pin_3)
- net ext_coil+ renamed out+
- no-connect marks 0 -> 1
Other:
- note added: "1, 2, 9, 10: Config 3: external coil (-) 4: GND 5: external coil (+) 6: out (+) 7: GND 8: out (-)"
- note added: "1: internal coil (mid) 2: GND 3: internal coil (-) 4: internal coil (+)"
- note removed: "Redundant connections to the coil via two small 1mm 2x3 connectors for improved reliability"
- moved on the sheet: H1, H2, H3, H4, J1

Commit message: CAD drawings, etc.
Other:
- note removed: "June 17, 2021"
- note removed: "Spectra Passive"
- company: (none) -> Document No. 2022013
- title: (none) -> XR Spectra Passive Board
Changed lines of the file:
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@@
 (kicad_sch (version 20211123) (generator eeschema)
   (paper "A4")
+  (title_block
+    (title "XR Spectra Passive Board")
+    (date "2022-12-22")
+    (rev "1.02")
+    (company "Document No. 2022013")
+  )
   (junction (at 110.49 60.96) (diameter 0) (color 0 0 0 0)
   )
@@
     (stroke (width 0) (type default) (color 0 0 0 0))
   )
-  (image (at 232.41 173.99) (scale 0.8)
+  (image (at 231.14 173.99) (scale 0.8)
     (data
       iVBORw0KGgoAAAANSUhEUgAABUAAAAB3CAYAAADCQeqJAAAABHNCSVQICAgIfAhkiAAAAAlwSFlz
@@
     (effects (font (size 1.27 1.27)) (justify left bottom))
   )
-  (text "June 17, 2021" (at 207.01 194.31 0)
-    (effects (font (size 1.27 1.27)) (justify left bottom))
-  )
-  (text "Spectra Passive" (at 187.96 190.5 0)
-    (effects (font (size 1.27 1.27)) (justify left bottom))
-  )
