File: hardware/base/base_3.3/base_3.3.sch (KiCad schematic (older format))
At the start: 6 parts, among them J1 Conn 1, J2 Conn 2

Commit message: Ok. Looks good.
Parts:
- added H5: single_pad_smd, cycfi_library:single-pad-5x3.5, symbol cycfi_library:single_pad_smd
Connections:
- net GND: now also H5.1
Changed lines of the file:
@@
 Text Label 4050 2550 0    50   ~ 0
 ic2
+$Comp
+L cycfi_library:single_pad_smd H5
+U 1 1 6112BC09
+P 4250 2850
+F 0 "H5" H 4250 2975 50  0000 L CNN
+F 1 "single_pad_smd" H 4250 3050 50  0001 C CNN
+F 2 "cycfi_library:single-pad-5x3.5" H 4250 2850 50  0001 C CNN
+F 3 "~" H 4250 2850 50  0001 C CNN
+	1    4250 2850
+	0    1    1    0
+$EndComp
+$Comp
+L power:GND #PWR03
+U 1 1 6112C732
+P 4000 2850
+F 0 "#PWR03" H 4000 2600 50  0001 C CNN
+F 1 "GND" H 4005 2677 50  0000 C CNN
+F 2 "" H 4000 2850 50  0001 C CNN
+F 3 "" H 4000 2850 50  0001 C CNN
+	1    4000 2850
+	1    0    0    -1
+$EndComp
+Wire Wire Line
+	4150 2850 4000 2850
 $EndSCHEMATC

Commit message: updates on grounding
Parts:
- added H6: single_pad_smd, cycfi_library:single-pad-5x3.5, symbol cycfi_library:single_pad_smd
- renumbered H2 to IC1, H4 to IC2, H1 to OC1, H3 to OC2
Connections:
- net GND: now also H6.1
Changed lines of the file:
@@
 1.0
 $Comp
-L cycfi_library:single_pad_smd H1
+L cycfi_library:single_pad_smd OC1
 U 1 1 61122909
 P 4250 1800
-F 0 "H1" H 4250 1925 50  0000 L CNN
+F 0 "OC1" H 4250 1925 50  0000 L CNN
 F 1 "single_pad_smd" H 4250 2000 50  0001 C CNN
 F 2 "cycfi_library:single-pad-3.5x2" H 4250 1800 50  0001 C CNN
@@
 $EndComp
 $Comp
-L cycfi_library:single_pad_smd H2
+L cycfi_library:single_pad_smd IC1
 U 1 1 61122FED
 P 4250 2050
-F 0 "H2" H 4250 2175 50  0000 L CNN
+F 0 "IC1" H 4250 2175 50  0000 L CNN
 F 1 "single_pad_smd" H 4250 2250 50  0001 C CNN
 F 2 "cycfi_library:single-pad-3.5x2" H 4250 2050 50  0001 C CNN
@@
 	2300 2450 2600 2450
 $Comp
-L cycfi_library:single_pad_smd H3
+L cycfi_library:single_pad_smd OC2
 U 1 1 6112FFAE
 P 4250 2300
-F 0 "H3" H 4250 2425 50  0000 L CNN
+F 0 "OC2" H 4250 2425 50  0000 L CNN
 F 1 "single_pad_smd" H 4250 2500 50  0001 C CNN
 F 2 "cycfi_library:single-pad-3.5x2" H 4250 2300 50  0001 C CNN
@@
 $EndComp
 $Comp
-L cycfi_library:single_pad_smd H4
+L cycfi_library:single_pad_smd IC2
 U 1 1 611302A2
 P 4250 2550
-F 0 "H4" H 4250 2675 50  0000 L CNN
+F 0 "IC2" H 4250 2675 50  0000 L CNN
 F 1 "single_pad_smd" H 4250 2750 50  0001 C CNN
 F 2 "cycfi_library:single-pad-3.5x2" H 4250 2550 50  0001 C CNN
@@
 U 1 1 6112BC09
 P 4250 2850
-F 0 "H5" H 4250 2975 50  0000 L CNN
+F 0 "H5" H 4250 2975 50  0001 L CNN
 F 1 "single_pad_smd" H 4250 3050 50  0001 C CNN
 F 2 "cycfi_library:single-pad-5x3.5" H 4250 2850 50  0001 C CNN
@@
 L power:GND #PWR03
 U 1 1 6112C732
-P 4000 2850
-F 0 "#PWR03" H 4000 2600 50  0001 C CNN
-F 1 "GND" H 4005 2677 50  0000 C CNN
-F 2 "" H 4000 2850 50  0001 C CNN
-F 3 "" H 4000 2850 50  0001 C CNN
-	1    4000 2850
-	1    0    0    -1
-$EndComp
-Wire Wire Line
-	4150 2850 4000 2850
+P 3850 2950
+F 0 "#PWR03" H 3850 2700 50  0001 C CNN
+F 1 "GND" H 3855 2777 50  0000 C CNN
+F 2 "" H 3850 2950 50  0001 C CNN
+F 3 "" H 3850 2950 50  0001 C CNN
+	1    3850 2950
+	1    0    0    -1
+$EndComp
+$Comp
+L cycfi_library:single_pad_smd H6
+U 1 1 6114C19E
+P 4250 3150
+F 0 "H6" H 4250 3275 50  0001 L CNN
+F 1 "single_pad_smd" H 4250 3350 50  0001 C CNN
+F 2 "cycfi_library:single-pad-5x3.5" H 4250 3150 50  0001 C CNN
+F 3 "~" H 4250 3150 50  0001 C CNN
+	1    4250 3150
+	0    1    1    0
+$EndComp
+Wire Wire Line
+	4150 2850 4050 2850
+Wire Wire Line
+	3850 2850 3850 2950
+Wire Wire Line
+	4150 3150 4050 3150
+Wire Wire Line
+	4050 3150 4050 2850
+Connection ~ 4050 2850
+Wire Wire Line
+	4050 2850 3850 2850
 $EndSCHEMATC

Commit message: base board xr-spectra v1.0
Parts:
- H5, H6: footprint cycfi_library:single-pad-5x3.5 -> cycfi_library:single-pad-3x2
- IC1, IC2, OC1, OC2: footprint cycfi_library:single-pad-3.5x2 -> cycfi_library:single-pad-2x2-th
Changed lines of the file:
@@
 F 0 "OC1" H 4250 1925 50  0000 L CNN
 F 1 "single_pad_smd" H 4250 2000 50  0001 C CNN
-F 2 "cycfi_library:single-pad-3.5x2" H 4250 1800 50  0001 C CNN
+F 2 "cycfi_library:single-pad-2x2-th" H 4250 1800 50  0001 C CNN
 F 3 "~" H 4250 1800 50  0001 C CNN
 	1    4250 1800
@@
 F 0 "IC1" H 4250 2175 50  0000 L CNN
 F 1 "single_pad_smd" H 4250 2250 50  0001 C CNN
-F 2 "cycfi_library:single-pad-3.5x2" H 4250 2050 50  0001 C CNN
+F 2 "cycfi_library:single-pad-2x2-th" H 4250 2050 50  0001 C CNN
 F 3 "~" H 4250 2050 50  0001 C CNN
 	1    4250 2050
@@
 F 0 "OC2" H 4250 2425 50  0000 L CNN
 F 1 "single_pad_smd" H 4250 2500 50  0001 C CNN
-F 2 "cycfi_library:single-pad-3.5x2" H 4250 2300 50  0001 C CNN
+F 2 "cycfi_library:single-pad-2x2-th" H 4250 2300 50  0001 C CNN
 F 3 "~" H 4250 2300 50  0001 C CNN
 	1    4250 2300
@@
 F 0 "IC2" H 4250 2675 50  0000 L CNN
 F 1 "single_pad_smd" H 4250 2750 50  0001 C CNN
-F 2 "cycfi_library:single-pad-3.5x2" H 4250 2550 50  0001 C CNN
+F 2 "cycfi_library:single-pad-2x2-th" H 4250 2550 50  0001 C CNN
 F 3 "~" H 4250 2550 50  0001 C CNN
 	1    4250 2550
@@
 F 0 "H5" H 4250 2975 50  0001 L CNN
 F 1 "single_pad_smd" H 4250 3050 50  0001 C CNN
-F 2 "cycfi_library:single-pad-5x3.5" H 4250 2850 50  0001 C CNN
+F 2 "cycfi_library:single-pad-3x2" H 4250 2850 50  0001 C CNN
 F 3 "~" H 4250 2850 50  0001 C CNN
 	1    4250 2850
@@
 L cycfi_library:single_pad_smd H6
 U 1 1 6114C19E
-P 4250 3150
-F 0 "H6" H 4250 3275 50  0001 L CNN
-F 1 "single_pad_smd" H 4250 3350 50  0001 C CNN
-F 2 "cycfi_library:single-pad-5x3.5" H 4250 3150 50  0001 C CNN
-F 3 "~" H 4250 3150 50  0001 C CNN
-	1    4250 3150
-	0    1    1    0
-$EndComp
-Wire Wire Line
-	4150 2850 4050 2850
+P 4250 3100
+F 0 "H6" H 4250 3225 50  0001 L CNN
+F 1 "single_pad_smd" H 4250 3300 50  0001 C CNN
+F 2 "cycfi_library:single-pad-3x2" H 4250 3100 50  0001 C CNN
+F 3 "~" H 4250 3100 50  0001 C CNN
+	1    4250 3100
+	0    1    1    0
+$EndComp
 Wire Wire Line
 	3850 2850 3850 2950
 Wire Wire Line
-	4150 3150 4050 3150
-Wire Wire Line
-	4050 3150 4050 2850
+	3850 2850 4050 2850
+Wire Wire Line
+	4050 2850 4050 3100
+Wire Wire Line
+	4050 3100 4150 3100
 Connection ~ 4050 2850
 Wire Wire Line
-	4050 2850 3850 2850
+	4050 2850 4150 2850
 $EndSCHEMATC

Commit message: take 1, redesign
Parts:
- removed H5, H6: single_pad_smd, cycfi_library:single-pad-3x2, symbol cycfi_library:single_pad_smd
- removed IC1, IC2, OC1, OC2: single_pad_smd, cycfi_library:single-pad-2x2-th, symbol cycfi_library:single_pad_smd
- added J3, J4: Conn_01x03, cycfi_library:xr2-coil-connector, symbol Connector_Generic:Conn_01x03
Connections:
- net GND: now also J3.1 (Pin_1), J4.1 (Pin_1)
- net ic2 renamed OC2
- net OC2: now also J4.2 (Pin_2)
- net oc1 renamed OC1
- net OC1: now also J3.2 (Pin_2)
- new net IC1: J3.3 (Pin_3), J4.3 (Pin_3)
Changed lines of the file:
@@
 1.0
-$Comp
-L cycfi_library:single_pad_smd OC1
-U 1 1 61122909
-P 4250 1800
-F 0 "OC1" H 4250 1925 50  0000 L CNN
-F 1 "single_pad_smd" H 4250 2000 50  0001 C CNN
-F 2 "cycfi_library:single-pad-2x2-th" H 4250 1800 50  0001 C CNN
-F 3 "~" H 4250 1800 50  0001 C CNN
-	1    4250 1800
-	0    1    1    0
-$EndComp
-$Comp
-L cycfi_library:single_pad_smd IC1
-U 1 1 61122FED
-P 4250 2050
-F 0 "IC1" H 4250 2175 50  0000 L CNN
-F 1 "single_pad_smd" H 4250 2250 50  0001 C CNN
-F 2 "cycfi_library:single-pad-2x2-th" H 4250 2050 50  0001 C CNN
-F 3 "~" H 4250 2050 50  0001 C CNN
-	1    4250 2050
-	0    1    1    0
-$EndComp
 $Comp
 L power:GND #PWR01
@@
 Wire Wire Line
 	2300 2450 2600 2450
-$Comp
-L cycfi_library:single_pad_smd OC2
-U 1 1 6112FFAE
-P 4250 2300
-F 0 "OC2" H 4250 2425 50  0000 L CNN
-F 1 "single_pad_smd" H 4250 2500 50  0001 C CNN
-F 2 "cycfi_library:single-pad-2x2-th" H 4250 2300 50  0001 C CNN
-F 3 "~" H 4250 2300 50  0001 C CNN
-	1    4250 2300
-	0    1    1    0
-$EndComp
-$Comp
-L cycfi_library:single_pad_smd IC2
-U 1 1 611302A2
-P 4250 2550
-F 0 "IC2" H 4250 2675 50  0000 L CNN
-F 1 "single_pad_smd" H 4250 2750 50  0001 C CNN
-F 2 "cycfi_library:single-pad-2x2-th" H 4250 2550 50  0001 C CNN
-F 3 "~" H 4250 2550 50  0001 C CNN
-	1    4250 2550
-	0    1    1    0
-$EndComp
 $Comp
 L Connector_Generic:Conn_02x03_Counter_Clockwise J1
@@
 	3550 2450 3550 2550
 Wire Wire Line
-	4150 1800 3900 1800
-Wire Wire Line
-	3900 1800 3900 1900
-Wire Wire Line
-	3900 1900 3550 1900
-Wire Wire Line
-	4150 2550 3900 2550
-Wire Wire Line
-	3900 2550 3900 2450
-Wire Wire Line
-	3900 2450 3550 2450
-Wire Wire Line
-	4150 2300 3950 2300
-Wire Wire Line
-	3950 2300 3950 2050
-Wire Wire Line
-	3950 2050 4150 2050
-Wire Wire Line
 	2950 2350 2800 2350
 Wire Wire Line
@@
 Wire Wire Line
 	2600 1900 2800 1900
-Text Label 4050 1800 0    50   ~ 0
-oc1
-Text Label 4050 2050 0    50   ~ 0
-ic1
-Text Label 4050 2300 0    50   ~ 0
-oc2
-Text Label 4050 2550 0    50   ~ 0
-ic2
 $Comp
-L cycfi_library:single_pad_smd H5
-U 1 1 6112BC09
-P 4250 2850
-F 0 "H5" H 4250 2975 50  0001 L CNN
-F 1 "single_pad_smd" H 4250 3050 50  0001 C CNN
-F 2 "cycfi_library:single-pad-3x2" H 4250 2850 50  0001 C CNN
-F 3 "~" H 4250 2850 50  0001 C CNN
-	1    4250 2850
-	0    1    1    0
-$EndComp
-$Comp
-L power:GND #PWR03
-U 1 1 6112C732
-P 3850 2950
-F 0 "#PWR03" H 3850 2700 50  0001 C CNN
-F 1 "GND" H 3855 2777 50  0000 C CNN
-F 2 "" H 3850 2950 50  0001 C CNN
-F 3 "" H 3850 2950 50  0001 C CNN
-	1    3850 2950
+L Connector_Generic:Conn_01x03 J3
+U 1 1 61509D32
+P 4300 1900
+F 0 "J3" H 4380 1942 50  0000 L CNN
+F 1 "Conn_01x03" H 4380 1851 50  0000 L CNN
+F 2 "cycfi_library:xr2-coil-connector" H 4300 1900 50  0001 C CNN
+F 3 "~" H 4300 1900 50  0001 C CNN
+	1    4300 1900
 	1    0    0    -1
 $EndComp
 $Comp
-L cycfi_library:single_pad_smd H6
-U 1 1 6114C19E
-P 4250 3100
-F 0 "H6" H 4250 3225 50  0001 L CNN
-F 1 "single_pad_smd" H 4250 3300 50  0001 C CNN
-F 2 "cycfi_library:single-pad-3x2" H 4250 3100 50  0001 C CNN
-F 3 "~" H 4250 3100 50  0001 C CNN
-	1    4250 3100
-	0    1    1    0
+L Connector_Generic:Conn_01x03 J4
+U 1 1 6150A3D8
+P 4300 2450
+F 0 "J4" H 4380 2492 50  0000 L CNN
+F 1 "Conn_01x03" H 4380 2401 50  0000 L CNN
+F 2 "cycfi_library:xr2-coil-connector" H 4300 2450 50  0001 C CNN
+F 3 "~" H 4300 2450 50  0001 C CNN
+	1    4300 2450
+	1    0    0    -1
+$EndComp
+$Comp
+L power:GND #PWR0101
+U 1 1 6150AFAE
+P 3800 2700
+F 0 "#PWR0101" H 3800 2450 50  0001 C CNN
+F 1 "GND" H 3805 2527 50  0000 C CNN
+F 2 "" H 3800 2700 50  0001 C CNN
+F 3 "" H 3800 2700 50  0001 C CNN
+	1    3800 2700
+	1    0    0    -1
 $EndComp
 Wire Wire Line
-	3850 2850 3850 2950
+	4100 2350 3800 2350
 Wire Wire Line
-	3850 2850 4050 2850
+	4100 1800 3800 1800
+Text Label 4100 1900 2    50   ~ 0
+OC1
+Text Label 4100 2000 2    50   ~ 0
+IC1
+Text Label 4100 2450 2    50   ~ 0
+OC2
+Text Label 4100 2550 2    50   ~ 0
+IC2
 Wire Wire Line
-	4050 2850 4050 3100
+	4100 2000 3900 2000
 Wire Wire Line
-	4050 3100 4150 3100
-Connection ~ 4050 2850
+	3900 2000 3900 2550
 Wire Wire Line
-	4050 2850 4150 2850
+	3900 2550 4100 2550
+Wire Wire Line
+	3800 1800 3800 2350
+Wire Wire Line
+	3800 2700 3800 2350
+Connection ~ 3800 2350
+Wire Wire Line
+	4100 1900 3550 1900
+Wire Wire Line
+	4100 2450 3550 2450
 $EndSCHEMATC
