File: hardware/base/base_3.3/base_3.3.kicad_pcb (KiCad board)
At the start: 2 copper layers, 77 x 17 mm, 9 parts, among them IC1 single_pad_smd, IC2 single_pad_smd, J1 Conn 1, J2 Conn 2

Commit message: take 1, redesign
Parts:
- removed GND (x2): single_pad_smd, cycfi_library:single-pad-3x2
- removed IC1, IC2, OC1, OC2: single_pad_smd, cycfi_library:single-pad-2x2-th
- added J3: Conn_01x03, cycfi_library:xr2-coil-connector, F.Cu at (140.5, 52.0)
- added J4: Conn_01x03, cycfi_library:xr2-coil-connector, F.Cu at (109.5, 58.5)
- moved J2 0.50 mm to (148.3, 55.2)
Connections:
- net /ic2 renamed /OC2
- net /oc1 renamed /OC1
Routing:
- net GND: track 78.3 -> 4.77 mm, vias 6 -> 2
- net /OC2: track 5.23 -> 41.9 mm
- net /ic1: track 34.3 -> 0.00 mm
- net /IC1: track 0.00 -> 30.4 mm
- net /OC1: track 45.5 -> 18.0 mm
Other:
- board text removed: "IC1"
- board text removed: "IC2"
- board text removed: "OC1"
- board text removed: "OC2"

Commit message: New scheme looking good.
Parts:
- moved J3 15.5 mm to (125.0, 52.0)
- moved J4 15.5 mm to (125.0, 58.5)
Routing:
- net /IC1: track 30.4 -> 10.2 mm
- net /OC1: track 18.0 -> 36.7 mm
- net /OC2: track 41.9 -> 27.3 mm
- net GND: track 4.77 -> 9.22 mm
Other:
- outline, holes or cut-outs redrawn

Commit message: updates for v1.01
Parts:
- moved J2 0.20 mm to (148.1, 55.2)
Changed lines of the file:
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@@
       (effects (font (size 1 1) (thickness 0.15)))
     )
-    (pad 3 thru_hole circle (at 2.54 0 180) (size 1.524 1.524) (drill 0.762) (layers *.Cu *.Mask F.SilkS)
+    (pad 3 thru_hole circle (at 2.54 0 180) (size 1.524 1.524) (drill 0.762) (layers *.Cu *.Mask)
       (net 4 /IC1))
     (pad 2 thru_hole circle (at 0 0 180) (size 1.524 1.524) (drill 0.762) (layers *.Cu *.Mask)
@@
       (effects (font (size 1 1) (thickness 0.15)))
     )
-    (fp_line (start 3.1 -1.6) (end -3.1 -1.6) (layer F.CrtYd) (width 0.05))
-    (fp_line (start 3.1 1.6) (end 3.1 -1.6) (layer F.CrtYd) (width 0.05))
-    (fp_line (start -3.1 1.6) (end 3.1 1.6) (layer F.CrtYd) (width 0.05))
-    (fp_line (start -3.1 -1.6) (end -3.1 1.6) (layer F.CrtYd) (width 0.05))
+    (fp_text user %R (at 0 0) (layer F.Fab)
+      (effects (font (size 1 1) (thickness 0.15)))
+    )
+    (fp_line (start 3.1 -1.7) (end -3.1 -1.7) (layer F.CrtYd) (width 0.05))
+    (fp_line (start 3.1 1.7) (end 3.1 -1.7) (layer F.CrtYd) (width 0.05))
+    (fp_line (start -3.1 1.7) (end 3.1 1.7) (layer F.CrtYd) (width 0.05))
+    (fp_line (start -3.1 -1.7) (end -3.1 1.7) (layer F.CrtYd) (width 0.05))
     (fp_line (start 1.15 1.4) (end 1.15 1.5) (layer F.SilkS) (width 0.12))
     (fp_line (start -1.15 1.4) (end -1.15 1.5) (layer F.SilkS) (width 0.12))
@@
     (fp_line (start -1.15 -1.5) (end 1.15 -1.5) (layer F.Fab) (width 0.1))
     (fp_line (start 1.15 1.5) (end -1.15 1.5) (layer F.Fab) (width 0.1))
-    (fp_circle (center -3.7 -1) (end -3.5 -1) (layer F.SilkS) (width 0.4))
-    (fp_text user %R (at 0 0) (layer F.Fab)
-      (effects (font (size 1 1) (thickness 0.15)))
-    )
     (pad 1 smd rect (at -1.9 -1 90) (size 2.4 0.56) (layers F.Cu F.Paste F.Mask)
       (net 1 GND))
@@
   )
   (module cycfi_library:pin_header_2x3p_1.00mm_smd_vertical (layer F.Cu)
-    (at 148.3 55.25 90)
+    (at 148.1 55.25 90)
     (descr "surface-mounted straight pin header, 2x03, 1.00mm pitch, double rows")
     (tags "Surface mounted pin header SMD 2x03 1.00mm double row")
@@
       (effects (font (size 1 1) (thickness 0.15)))
     )
-    (fp_line (start 3.1 -1.6) (end -3.1 -1.6) (layer F.CrtYd) (width 0.05))
-    (fp_line (start 3.1 1.6) (end 3.1 -1.6) (layer F.CrtYd) (width 0.05))
-    (fp_line (start -3.1 1.6) (end 3.1 1.6) (layer F.CrtYd) (width 0.05))
-    (fp_line (start -3.1 -1.6) (end -3.1 1.6) (layer F.CrtYd) (width 0.05))
+    (fp_text user %R (at 0 0) (layer F.Fab)
+      (effects (font (size 1 1) (thickness 0.15)))
+    )
+    (fp_line (start 3.1 -1.7) (end -3.1 -1.7) (layer F.CrtYd) (width 0.05))
+    (fp_line (start 3.1 1.7) (end 3.1 -1.7) (layer F.CrtYd) (width 0.05))
+    (fp_line (start -3.1 1.7) (end 3.1 1.7) (layer F.CrtYd) (width 0.05))
+    (fp_line (start -3.1 -1.7) (end -3.1 1.7) (layer F.CrtYd) (width 0.05))
     (fp_line (start 1.15 1.4) (end 1.15 1.5) (layer F.SilkS) (width 0.12))
     (fp_line (start -1.15 1.4) (end -1.15 1.5) (layer F.SilkS) (width 0.12))
@@
     (fp_line (start -1.15 -1.5) (end 1.15 -1.5) (layer F.Fab) (width 0.1))
     (fp_line (start 1.15 1.5) (end -1.15 1.5) (layer F.Fab) (width 0.1))
-    (fp_circle (center -3.7 -1) (end -3.5 -1) (layer F.SilkS) (width 0.4))
-    (fp_text user %R (at 0 0) (layer F.Fab)
-      (effects (font (size 1 1) (thickness 0.15)))
-    )
     (pad 1 smd rect (at -1.9 -1 90) (size 2.4 0.56) (layers F.Cu F.Paste F.Mask)
       (net 1 GND))

Commit message: Update from Solidworks
Routing:
- net /OC1: track 36.7 -> 37.8 mm
Other:
- outline, holes or cut-outs redrawn
