File: hardware/base/base_3.5/base_3.5.kicad_sch (KiCad schematic)
At the start: 7 parts, among them IC1 single_pad, IC2 single_pad, J1 conn_2x2

Commit message: 3.5" PCB layout
Parts:
- added H1, H2: MountingHole, cycfi_library:hole_3mm, symbol Mechanical:MountingHole
- H5, H6: footprint xr_spectra_library:rail_slot_3.3 -> xr_spectra_library:rail_slot_3.5
Other:
- note added: "Mounting Holes"
Changed lines of the file:
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@@
     )
+  )
+  (text "Mounting Holes" (at 191.77 88.9 0)
+    (effects (font (size 1.27 1.27)) (justify left bottom))
   )
   (text "Spectra Passive" (at 187.96 190.5 0)
@@
       (effects (font (size 1.27 1.27)) hide)
     )
-    (property "Footprint" "xr_spectra_library:rail_slot_3.3" (id 2) (at 172.72 97.79 0)
+    (property "Footprint" "xr_spectra_library:rail_slot_3.5" (id 2) (at 172.72 97.79 0)
       (effects (font (size 1.27 1.27)) hide)
     )
@@
       (effects (font (size 1.27 1.27)) hide)
     )
-    (property "Footprint" "xr_spectra_library:rail_slot_3.3" (id 2) (at 172.72 104.14 0)
+    (property "Footprint" "xr_spectra_library:rail_slot_3.5" (id 2) (at 172.72 104.14 0)
       (effects (font (size 1.27 1.27)) hide)
     )
@@
     (pin "4")
   )
+  (symbol (lib_id "Mechanical:MountingHole") (at 198.12 82.55 0) (unit 1)
+    (in_bom yes) (on_board yes) (fields_autoplaced)
+    (property "Reference" "H2" (id 0) (at 200.66 82.9838 0)
+      (effects (font (size 1.27 1.27)) (justify left))
+    )
+    (property "Value" "MountingHole" (id 1) (at 200.66 84.2522 0)
+      (effects (font (size 1.27 1.27)) (justify left) hide)
+    )
+    (property "Footprint" "cycfi_library:hole_3mm" (id 2) (at 198.12 82.55 0)
+      (effects (font (size 1.27 1.27)) hide)
+    )
+    (property "Datasheet" "~" (id 3) (at 198.12 82.55 0)
+      (effects (font (size 1.27 1.27)) hide)
+    )
+  )
+  (symbol (lib_id "Mechanical:MountingHole") (at 198.12 76.2 0) (unit 1)
+    (in_bom yes) (on_board yes) (fields_autoplaced)
+    (property "Reference" "H1" (id 0) (at 200.66 76.6338 0)
+      (effects (font (size 1.27 1.27)) (justify left))
+    )
+    (property "Value" "MountingHole" (id 1) (at 200.66 77.9022 0)
+      (effects (font (size 1.27 1.27)) (justify left) hide)
+    )
+    (property "Footprint" "cycfi_library:hole_3mm" (id 2) (at 198.12 76.2 0)
+      (effects (font (size 1.27 1.27)) hide)
+    )
+    (property "Datasheet" "~" (id 3) (at 198.12 76.2 0)
+      (effects (font (size 1.27 1.27)) hide)
+    )
+  )
   (sheet_instances
     (path "/" (page "1"))
@@
       (reference "#PWR03") (unit 1) (value "GND") (footprint "")
     )
+    (path "/f74eb612-4697-4cb4-afe4-9f94828b954d"
+      (reference "H1") (unit 1) (value "MountingHole") (footprint "cycfi_library:hole_3mm")
+    )
+    (path "/f52f1267-ef72-4576-80d0-5917f82db729"
+      (reference "H2") (unit 1) (value "MountingHole") (footprint "cycfi_library:hole_3mm")
+    )
     (path "/00000000-0000-0000-0000-00006112bc09"
-      (reference "H5") (unit 1) (value "single_pad") (footprint "xr_spectra_library:rail_slot_3.3")
+      (reference "H5") (unit 1) (value "single_pad") (footprint "xr_spectra_library:rail_slot_3.5")
     )
     (path "/00000000-0000-0000-0000-00006114c19e"
-      (reference "H6") (unit 1) (value "single_pad") (footprint "xr_spectra_library:rail_slot_3.3")
+      (reference "H6") (unit 1) (value "single_pad") (footprint "xr_spectra_library:rail_slot_3.5")
     )
     (path "/00000000-0000-0000-0000-000061122fed"

Commit message: PCB layout 3.5"
Parts:
- H1, H2: footprint cycfi_library:hole_3mm -> (none)
- renumbered OC1 to IC1, OC2 to IC2, IC1 to OC1, IC2 to OC2
Connections:
- net inner_coil renamed middle_coil
Changed lines of the file:
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@@
     (stroke (width 0) (type default) (color 0 0 0 0))
   )
-  (polyline (pts (xy 123.825 86.995) (xy 123.825 100.965))
+  (polyline (pts (xy 123.19 87.63) (xy 123.19 101.6))
     (stroke (width 0) (type default) (color 0 0 0 0))
   )
@@
     (stroke (width 0) (type default) (color 0 0 0 0))
   )
-  (polyline (pts (xy 123.825 86.995) (xy 151.765 86.995))
+  (polyline (pts (xy 123.19 87.63) (xy 152.4 87.63))
     (stroke (width 0) (type default) (color 0 0 0 0))
   )
@@
     (stroke (width 0) (type default) (color 0 0 0 0))
   )
-  (polyline (pts (xy 151.765 100.965) (xy 123.825 100.965))
+  (polyline (pts (xy 152.4 101.6) (xy 123.19 101.6))
     (stroke (width 0) (type default) (color 0 0 0 0))
   )
@@
     (stroke (width 0) (type default) (color 0 0 0 0))
   )
-  (polyline (pts (xy 151.765 86.995) (xy 151.765 100.965))
+  (polyline (pts (xy 152.4 87.63) (xy 152.4 101.6))
     (stroke (width 0) (type default) (color 0 0 0 0))
   )
@@
     )
   )
-  (text "Mounting Holes" (at 191.77 88.9 0)
-    (effects (font (size 1.27 1.27)) (justify left bottom))
-  )
   (text "Spectra Passive" (at 187.96 190.5 0)
     (effects (font (size 1.27 1.27)) (justify left bottom))
@@
     (effects (font (size 1.27 1.27)) (justify left bottom))
   )
+  (text "Mounting Holes" (at 193.04 93.98 0)
+    (effects (font (size 1.27 1.27)) (justify left bottom))
+  )
   (text "June 17, 2021" (at 207.01 194.31 0)
     (effects (font (size 1.27 1.27)) (justify left bottom))
@@
     (effects (font (size 1.27 1.27)) (justify left bottom))
   )
-  (global_label "inner_coil" (shape input) (at 133.35 71.12 180) (fields_autoplaced)
+  (global_label "middle_coil" (shape input) (at 133.35 71.12 180) (fields_autoplaced)
     (effects (font (size 1.27 1.27)) (justify right))
-    (property "Intersheet References" "${INTERSHEET_REFS}" (id 0) (at 121.7729 71.0406 0)
+    (property "Intersheet References" "${INTERSHEET_REFS}" (id 0) (at 120.2006 71.0406 0)
       (effects (font (size 1.27 1.27)) (justify right) hide)
     )
@@
   (symbol (lib_id "cycfi_library:single_pad") (at 172.72 71.12 270) (unit 1)
     (in_bom yes) (on_board yes)
-    (property "Reference" "OC1" (id 0) (at 175.895 71.12 90)
+    (property "Reference" "IC1" (id 0) (at 175.895 71.12 90)
       (effects (font (size 1.27 1.27)) (justify left))
     )
@@
   (symbol (lib_id "cycfi_library:single_pad") (at 172.72 77.47 270) (unit 1)
     (in_bom yes) (on_board yes)
-    (property "Reference" "IC1" (id 0) (at 175.895 77.47 90)
+    (property "Reference" "OC1" (id 0) (at 175.895 77.47 90)
       (effects (font (size 1.27 1.27)) (justify left))
     )
@@
   (symbol (lib_id "cycfi_library:single_pad") (at 172.72 90.17 270) (unit 1)
     (in_bom yes) (on_board yes)
-    (property "Reference" "OC2" (id 0) (at 175.895 90.17 90)
+    (property "Reference" "IC2" (id 0) (at 175.895 90.17 90)
       (effects (font (size 1.27 1.27)) (justify left))
     )
@@
   (symbol (lib_id "cycfi_library:single_pad") (at 172.72 83.82 270) (unit 1)
     (in_bom yes) (on_board yes)
-    (property "Reference" "IC2" (id 0) (at 175.895 83.82 90)
+    (property "Reference" "OC2" (id 0) (at 175.895 83.82 90)
       (effects (font (size 1.27 1.27)) (justify left))
     )
@@
     )
     (pin "1")
+  )
+  (symbol (lib_id "Mechanical:MountingHole") (at 199.39 81.28 0) (unit 1)
+    (in_bom yes) (on_board yes) (fields_autoplaced)
+    (property "Reference" "H1" (id 0) (at 201.93 80.4453 0)
+      (effects (font (size 1.27 1.27)) (justify left))
+    )
+    (property "Value" "MountingHole" (id 1) (at 201.93 82.9822 0)
+      (effects (font (size 1.27 1.27)) (justify left) hide)
+    )
+    (property "Footprint" "" (id 2) (at 199.39 81.28 0)
+      (effects (font (size 1.27 1.27)) hide)
+    )
+    (property "Datasheet" "~" (id 3) (at 199.39 81.28 0)
+      (effects (font (size 1.27 1.27)) hide)
+    )
   )
   (symbol (lib_id "Connector_Generic:Conn_02x02_Counter_Clockwise") (at 140.97 71.12 0) (unit 1)
@@
     (pin "4")
   )
-  (symbol (lib_id "Mechanical:MountingHole") (at 198.12 82.55 0) (unit 1)
+  (symbol (lib_id "Mechanical:MountingHole") (at 199.39 87.63 0) (unit 1)
     (in_bom yes) (on_board yes) (fields_autoplaced)
-    (property "Reference" "H2" (id 0) (at 200.66 82.9838 0)
-      (effects (font (size 1.27 1.27)) (justify left))
-    )
-    (property "Value" "MountingHole" (id 1) (at 200.66 84.2522 0)
+    (property "Reference" "H2" (id 0) (at 201.93 88.0638 0)
+      (effects (font (size 1.27 1.27)) (justify left))
+    )
+    (property "Value" "MountingHole" (id 1) (at 201.93 89.3322 0)
       (effects (font (size 1.27 1.27)) (justify left) hide)
     )
-    (property "Footprint" "cycfi_library:hole_3mm" (id 2) (at 198.12 82.55 0)
-      (effects (font (size 1.27 1.27)) hide)
-    )
-    (property "Datasheet" "~" (id 3) (at 198.12 82.55 0)
-      (effects (font (size 1.27 1.27)) hide)
-    )
-  )
-  (symbol (lib_id "Mechanical:MountingHole") (at 198.12 76.2 0) (unit 1)
-    (in_bom yes) (on_board yes) (fields_autoplaced)
-    (property "Reference" "H1" (id 0) (at 200.66 76.6338 0)
-      (effects (font (size 1.27 1.27)) (justify left))
-    )
-    (property "Value" "MountingHole" (id 1) (at 200.66 77.9022 0)
-      (effects (font (size 1.27 1.27)) (justify left) hide)
-    )
-    (property "Footprint" "cycfi_library:hole_3mm" (id 2) (at 198.12 76.2 0)
-      (effects (font (size 1.27 1.27)) hide)
-    )
-    (property "Datasheet" "~" (id 3) (at 198.12 76.2 0)
+    (property "Footprint" "" (id 2) (at 199.39 87.63 0)
+      (effects (font (size 1.27 1.27)) hide)
+    )
+    (property "Datasheet" "~" (id 3) (at 199.39 87.63 0)
       (effects (font (size 1.27 1.27)) hide)
     )
@@
       (reference "#PWR03") (unit 1) (value "GND") (footprint "")
     )
-    (path "/f74eb612-4697-4cb4-afe4-9f94828b954d"
-      (reference "H1") (unit 1) (value "MountingHole") (footprint "cycfi_library:hole_3mm")
-    )
-    (path "/f52f1267-ef72-4576-80d0-5917f82db729"
-      (reference "H2") (unit 1) (value "MountingHole") (footprint "cycfi_library:hole_3mm")
+    (path "/6f1beb86-67e1-46bf-8c2b-6d1e1485d5c0"
+      (reference "H1") (unit 1) (value "MountingHole") (footprint "")
+    )
+    (path "/b90f2dfd-9639-4bac-9825-9f33089900c6"
+      (reference "H2") (unit 1) (value "MountingHole") (footprint "")
     )
     (path "/00000000-0000-0000-0000-00006112bc09"
@@
       (reference "H6") (unit 1) (value "single_pad") (footprint "xr_spectra_library:rail_slot_3.5")
     )
-    (path "/00000000-0000-0000-0000-000061122fed"
+    (path "/00000000-0000-0000-0000-000061122909"
       (reference "IC1") (unit 1) (value "single_pad") (footprint "cycfi_library:single-pad-1.6x1.6_circular")
     )
-    (path "/00000000-0000-0000-0000-0000611302a2"
+    (path "/00000000-0000-0000-0000-00006112ffae"
       (reference "IC2") (unit 1) (value "single_pad") (footprint "cycfi_library:single-pad-1.6x1.6_circular")
     )
@@
       (reference "J1") (unit 1) (value "conn_2x2") (footprint "cycfi_library:pin_header_2x2p_2.00mm_smd_vertical")
     )
-    (path "/00000000-0000-0000-0000-000061122909"
+    (path "/00000000-0000-0000-0000-000061122fed"
       (reference "OC1") (unit 1) (value "single_pad") (footprint "cycfi_library:single-pad-1.6x1.6_circular")
     )
-    (path "/00000000-0000-0000-0000-00006112ffae"
+    (path "/00000000-0000-0000-0000-0000611302a2"
       (reference "OC2") (unit 1) (value "single_pad") (footprint "cycfi_library:single-pad-1.6x1.6_circular")
     )

Commit message: 3.5" and 3.3" good to go
Parts:
- H1, H2: footprint (none) -> cycfi_library:hole_3mm
Changed lines of the file:
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@@
       (effects (font (size 1.27 1.27)) (justify left) hide)
     )
-    (property "Footprint" "" (id 2) (at 199.39 81.28 0)
+    (property "Footprint" "cycfi_library:hole_3mm" (id 2) (at 199.39 81.28 0)
       (effects (font (size 1.27 1.27)) hide)
     )
@@
       (effects (font (size 1.27 1.27)) (justify left) hide)
     )
-    (property "Footprint" "" (id 2) (at 199.39 87.63 0)
+    (property "Footprint" "cycfi_library:hole_3mm" (id 2) (at 199.39 87.63 0)
       (effects (font (size 1.27 1.27)) hide)
     )
@@
     )
     (path "/6f1beb86-67e1-46bf-8c2b-6d1e1485d5c0"
-      (reference "H1") (unit 1) (value "MountingHole") (footprint "")
+      (reference "H1") (unit 1) (value "MountingHole") (footprint "cycfi_library:hole_3mm")
     )
     (path "/b90f2dfd-9639-4bac-9825-9f33089900c6"
-      (reference "H2") (unit 1) (value "MountingHole") (footprint "")
+      (reference "H2") (unit 1) (value "MountingHole") (footprint "cycfi_library:hole_3mm")
     )
     (path "/00000000-0000-0000-0000-00006112bc09"
