File: hardware/bobbin/bobbin_top_4.0/bobbin_top_4.0.kicad_sch (KiCad schematic)
At the start: 5 parts, among them J1 OC, J2 OC, J3 IC, J4 IC

Commit message: Bobbin-top done
Parts:
- removed J1, J2: OC, cycfi_library:single-pad-1.52x1.52-th, symbol Connector_Generic:Conn_01x01
- removed J3, J4: IC, cycfi_library:single-pad-1.52x1.52-th, symbol Connector_Generic:Conn_01x01
Changed lines of the file:
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@@
     (stroke (width 0) (type default) (color 0 0 0 0))
-  )
-  (label "IC" (at 147.32 71.12 180)
-    (effects (font (size 1.27 1.27)) (justify right bottom))
-  )
-  (label "OC" (at 147.32 60.96 180)
-    (effects (font (size 1.27 1.27)) (justify right bottom))
-  )
-  (label "OC" (at 147.32 55.88 180)
-    (effects (font (size 1.27 1.27)) (justify right bottom))
-  )
-  (label "IC" (at 147.32 66.04 180)
-    (effects (font (size 1.27 1.27)) (justify right bottom))
-  )
-  (symbol (lib_id "Connector_Generic:Conn_01x01") (at 152.4 60.96 0) (unit 1)
-    (in_bom yes) (on_board yes)
-    (property "Reference" "J2" (id 0) (at 154.432 59.8932 0)
-      (effects (font (size 1.27 1.27)) (justify left))
-    )
-    (property "Value" "OC" (id 1) (at 154.432 62.2046 0)
-      (effects (font (size 1.27 1.27)) (justify left))
-    )
-    (property "Footprint" "cycfi_library:single-pad-1.52x1.52-th" (id 2) (at 152.4 60.96 0)
-      (effects (font (size 1.27 1.27)) hide)
-    )
-    (property "Datasheet" "~" (id 3) (at 152.4 60.96 0)
-      (effects (font (size 1.27 1.27)) hide)
-    )
-    (pin "1")
   )
   (symbol (lib_id "power:GND") (at 140.97 83.82 0) (unit 1)
@@
     (pin "1")
   )
-  (symbol (lib_id "Connector_Generic:Conn_01x01") (at 152.4 55.88 0) (unit 1)
-    (in_bom yes) (on_board yes)
-    (property "Reference" "J1" (id 0) (at 154.432 54.8132 0)
-      (effects (font (size 1.27 1.27)) (justify left))
-    )
-    (property "Value" "OC" (id 1) (at 154.432 57.1246 0)
-      (effects (font (size 1.27 1.27)) (justify left))
-    )
-    (property "Footprint" "cycfi_library:single-pad-1.52x1.52-th" (id 2) (at 152.4 55.88 0)
-      (effects (font (size 1.27 1.27)) hide)
-    )
-    (property "Datasheet" "~" (id 3) (at 152.4 55.88 0)
-      (effects (font (size 1.27 1.27)) hide)
-    )
-    (pin "1")
-  )
-  (symbol (lib_id "Connector_Generic:Conn_01x01") (at 152.4 71.12 0) (unit 1)
-    (in_bom yes) (on_board yes)
-    (property "Reference" "J4" (id 0) (at 154.432 70.0532 0)
-      (effects (font (size 1.27 1.27)) (justify left))
-    )
-    (property "Value" "IC" (id 1) (at 154.432 72.3646 0)
-      (effects (font (size 1.27 1.27)) (justify left))
-    )
-    (property "Footprint" "cycfi_library:single-pad-1.52x1.52-th" (id 2) (at 152.4 71.12 0)
-      (effects (font (size 1.27 1.27)) hide)
-    )
-    (property "Datasheet" "~" (id 3) (at 152.4 71.12 0)
-      (effects (font (size 1.27 1.27)) hide)
-    )
-    (pin "1")
-  )
-  (symbol (lib_id "Connector_Generic:Conn_01x01") (at 152.4 66.04 0) (unit 1)
-    (in_bom yes) (on_board yes)
-    (property "Reference" "J3" (id 0) (at 154.432 64.9732 0)
-      (effects (font (size 1.27 1.27)) (justify left))
-    )
-    (property "Value" "IC" (id 1) (at 154.432 67.2846 0)
-      (effects (font (size 1.27 1.27)) (justify left))
-    )
-    (property "Footprint" "cycfi_library:single-pad-1.52x1.52-th" (id 2) (at 152.4 66.04 0)
-      (effects (font (size 1.27 1.27)) hide)
-    )
-    (property "Datasheet" "~" (id 3) (at 152.4 66.04 0)
-      (effects (font (size 1.27 1.27)) hide)
-    )
-    (pin "1")
-  )
   (sheet_instances
     (path "/" (page "1"))
@@
       (reference "H1") (unit 1) (value "single_pad") (footprint "xr_spectra_library:rail_slot_4.0")
     )
-    (path "/9ed5f09d-f428-462b-978c-7a9dd8637c06"
-      (reference "J1") (unit 1) (value "OC") (footprint "cycfi_library:single-pad-1.52x1.52-th")
-    )
-    (path "/00000000-0000-0000-0000-00006150ec9c"
-      (reference "J2") (unit 1) (value "OC") (footprint "cycfi_library:single-pad-1.52x1.52-th")
-    )
-    (path "/f226d0fa-6fa6-4f46-99cf-6860d539dd2c"
-      (reference "J3") (unit 1) (value "IC") (footprint "cycfi_library:single-pad-1.52x1.52-th")
-    )
-    (path "/a996384d-e545-45bd-921b-60bec151aabf"
-      (reference "J4") (unit 1) (value "IC") (footprint "cycfi_library:single-pad-1.52x1.52-th")
-    )
   )
