File: hardware/base/base_board_60/base_board_60.kicad_pcb (KiCad board)
At the start: 2 copper layers, 69 x 18 mm, 9 parts, among them IC1 single_pad, IC2 single_pad, J1 conn_2x2

Commit message: Minor tweaks after renames
Other:
- board text added: "OC1/2"
- board text removed: "X"
Changed lines of the file:
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@@
     (descr "Through hole straight pin header, 1x01, 2.54mm pitch, single row")
     (tags "Through hole pin header THT 1x01 2.54mm single row")
-    (property "Sheetfile" "File: base_3.3.kicad_sch")
+    (property "Sheetfile" "File: base_board_60.kicad_sch")
     (property "Sheetname" "")
     (attr through_hole)
@@
     (descr "Through hole straight pin header, 1x01, 2.54mm pitch, single row")
     (tags "Through hole pin header THT 1x01 2.54mm single row")
-    (property "Sheetfile" "File: base_3.3.kicad_sch")
+    (property "Sheetfile" "File: base_board_60.kicad_sch")
     (property "Sheetname" "")
     (attr through_hole)
@@
     (descr "Through hole straight pin header, 1x01, 2.54mm pitch, single row")
     (tags "Through hole pin header THT 1x01 2.54mm single row")
-    (property "Sheetfile" "File: base_3.3.kicad_sch")
+    (property "Sheetfile" "File: base_board_60.kicad_sch")
     (property "Sheetname" "")
     (attr through_hole)
@@
     (descr "Through hole straight pin header, 1x01, 2.54mm pitch, single row")
     (tags "Through hole pin header THT 1x01 2.54mm single row")
-    (property "Sheetfile" "File: base_3.3.kicad_sch")
+    (property "Sheetfile" "File: base_board_60.kicad_sch")
     (property "Sheetname" "")
     (attr through_hole)
@@
     (descr "surface-mounted straight pin socket, 2x2, 2.00mm pitch, double rows")
     (tags "Surface mounted pin header SMD 2x2 200mm double row")
-    (property "Sheetfile" "File: base_3.3.kicad_sch")
+    (property "Sheetfile" "File: base_board_60.kicad_sch")
     (property "Sheetname" "")
     (attr smd)
@@
     (effects (font (size 0.8 0.8) (thickness 0.1)) (justify mirror))
   )
-  (gr_text "X" (at 121.088095 51.95 180) (layer "B.SilkS")
+  (gr_text "OC1/2" (at 119.45 52.05 180) (layer "B.SilkS")
     (effects (font (size 0.8 0.8) (thickness 0.1)) (justify mirror))
   )
