File: hardware/base/base_board_60/base_board_60.kicad_sch (KiCad schematic)
At the start: 5 parts, among them IC1 single_pad, IC2 single_pad, J1 conn_2x2

Commit message: Minor tweaks after renames
Other:
- company: (none) -> Document No. 2024005
- title: (none) -> XR Spectra Base Board 60
Changed lines of the file:
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@@
 (kicad_sch (version 20211123) (generator eeschema)
   (paper "A4")
+  (title_block
+    (title "XR Spectra Base Board 60")
+    (date "2024-12-01")
+    (rev "v3.0")
+    (company "Document No. 2024005")
+  )
   (junction (at 166.37 77.47) (diameter 0) (color 0 0 0 0)
   )
