File: hardware/base_board/base_board_82/base_board_82.kicad_sch (KiCad schematic)
At the start: 9 parts, among them IC1 single_pad, IC2 single_pad, J1 conn_2x2

Commit message: base_boards 60, 70 and 82
Parts:
- removed H1, H2: MountingHole, cycfi_library:hole_3mm, symbol Mechanical:MountingHole
- removed H5, H6: single_pad, xr_spectra_library:rail_slot_3.5, symbol cycfi_library:single_pad
- IC1, IC2, OC1, OC2: footprint cycfi_library:single-pad-1.6x1.6_circular -> Connector_PinHeader_2.54mm:PinHeader_1x01_P2.54mm_Vertical
Other:
- note removed: "Mounting Holes"
- company: (none) -> Document No. 2024007
- title: (none) -> XR Spectra Base Board 82
Changed lines of the file:
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@@
 (kicad_sch (version 20211123) (generator eeschema)
   (paper "A4")
-  (junction (at 167.64 97.79) (diameter 0) (color 0 0 0 0)
+  (title_block
+    (title "XR Spectra Base Board 82")
+    (date "2024-12-02")
+    (rev "v3.0")
+    (company "Document No. 2024007")
   )
   (junction (at 166.37 77.47) (diameter 0) (color 0 0 0 0)
@@
     (stroke (width 0) (type default) (color 0 0 0 0))
   )
-  (wire (pts (xy 170.18 97.79) (xy 167.64 97.79))
-    (stroke (width 0) (type default) (color 0 0 0 0))
-  )
   (wire (pts (xy 130.81 73.66) (xy 135.89 73.66))
     (stroke (width 0) (type default) (color 0 0 0 0))
@@
     (stroke (width 0) (type default) (color 0 0 0 0))
   )
-  (wire (pts (xy 167.64 104.14) (xy 167.64 97.79))
-    (stroke (width 0) (type default) (color 0 0 0 0))
-  )
   (wire (pts (xy 148.59 73.66) (xy 158.75 73.66))
     (stroke (width 0) (type default) (color 0 0 0 0))
@@
     (stroke (width 0) (type default) (color 0 0 0 0))
   )
-  (wire (pts (xy 162.56 97.79) (xy 162.56 100.33))
-    (stroke (width 0) (type default) (color 0 0 0 0))
-  )
-  (wire (pts (xy 170.18 104.14) (xy 167.64 104.14))
-    (stroke (width 0) (type default) (color 0 0 0 0))
-  )
   (polyline (pts (xy 152.4 101.6) (xy 123.19 101.6))
-    (stroke (width 0) (type default) (color 0 0 0 0))
-  )
-  (wire (pts (xy 167.64 97.79) (xy 162.56 97.79))
     (stroke (width 0) (type default) (color 0 0 0 0))
   )
@@
     (effects (font (size 1.27 1.27)) (justify left bottom))
   )
-  (text "Mounting Holes" (at 193.04 93.98 0)
-    (effects (font (size 1.27 1.27)) (justify left bottom))
-  )
   (text "June 17, 2021" (at 207.01 194.31 0)
     (effects (font (size 1.27 1.27)) (justify left bottom))
@@
       (effects (font (size 1.27 1.27)) hide)
     )
-    (property "Footprint" "cycfi_library:single-pad-1.6x1.6_circular" (id 2) (at 172.72 71.12 0)
+    (property "Footprint" "Connector_PinHeader_2.54mm:PinHeader_1x01_P2.54mm_Vertical" (id 2) (at 172.72 71.12 0)
       (effects (font (size 1.27 1.27)) hide)
     )
@@
       (effects (font (size 1.27 1.27)) hide)
     )
-    (property "Footprint" "cycfi_library:single-pad-1.6x1.6_circular" (id 2) (at 172.72 77.47 0)
+    (property "Footprint" "Connector_PinHeader_2.54mm:PinHeader_1x01_P2.54mm_Vertical" (id 2) (at 172.72 77.47 0)
       (effects (font (size 1.27 1.27)) hide)
     )
@@
     )
     (property "Datasheet" "~" (id 3) (at 130.81 74.93 0)
-      (effects (font (size 1.27 1.27)) hide)
-    )
-    (pin "1")
-  )
-  (symbol (lib_id "cycfi_library:single_pad") (at 172.72 97.79 270) (unit 1)
-    (in_bom yes) (on_board yes)
-    (property "Reference" "H5" (id 0) (at 175.895 97.79 0)
-      (effects (font (size 1.27 1.27)) (justify left) hide)
-    )
-    (property "Value" "single_pad" (id 1) (at 177.8 97.79 0)
-      (effects (font (size 1.27 1.27)) hide)
-    )
-    (property "Footprint" "xr_spectra_library:rail_slot_3.5" (id 2) (at 172.72 97.79 0)
-      (effects (font (size 1.27 1.27)) hide)
-    )
-    (property "Datasheet" "~" (id 3) (at 172.72 97.79 0)
-      (effects (font (size 1.27 1.27)) hide)
-    )
-    (pin "1")
-  )
-  (symbol (lib_id "power:GND") (at 162.56 100.33 0) (unit 1)
-    (in_bom yes) (on_board yes)
-    (property "Reference" "#PWR03" (id 0) (at 162.56 106.68 0)
-      (effects (font (size 1.27 1.27)) hide)
-    )
-    (property "Value" "GND" (id 1) (at 162.687 104.7242 0))
-    (property "Footprint" "" (id 2) (at 162.56 100.33 0)
-      (effects (font (size 1.27 1.27)) hide)
-    )
-    (property "Datasheet" "" (id 3) (at 162.56 100.33 0)
       (effects (font (size 1.27 1.27)) hide)
     )
@@
       (effects (font (size 1.27 1.27)) hide)
     )
-    (property "Footprint" "cycfi_library:single-pad-1.6x1.6_circular" (id 2) (at 172.72 90.17 0)
+    (property "Footprint" "Connector_PinHeader_2.54mm:PinHeader_1x01_P2.54mm_Vertical" (id 2) (at 172.72 90.17 0)
       (effects (font (size 1.27 1.27)) hide)
     )
@@
       (effects (font (size 1.27 1.27)) hide)
     )
-    (property "Footprint" "cycfi_library:single-pad-1.6x1.6_circular" (id 2) (at 172.72 83.82 0)
+    (property "Footprint" "Connector_PinHeader_2.54mm:PinHeader_1x01_P2.54mm_Vertical" (id 2) (at 172.72 83.82 0)
       (effects (font (size 1.27 1.27)) hide)
     )
     (property "Datasheet" "~" (id 3) (at 172.72 83.82 0)
-      (effects (font (size 1.27 1.27)) hide)
-    )
-    (pin "1")
-  )
-  (symbol (lib_id "cycfi_library:single_pad") (at 172.72 104.14 270) (unit 1)
-    (in_bom yes) (on_board yes)
-    (property "Reference" "H6" (id 0) (at 175.895 104.14 0)
-      (effects (font (size 1.27 1.27)) (justify left) hide)
-    )
-    (property "Value" "single_pad" (id 1) (at 177.8 104.14 0)
-      (effects (font (size 1.27 1.27)) hide)
-    )
-    (property "Footprint" "xr_spectra_library:rail_slot_3.5" (id 2) (at 172.72 104.14 0)
-      (effects (font (size 1.27 1.27)) hide)
-    )
-    (property "Datasheet" "~" (id 3) (at 172.72 104.14 0)
       (effects (font (size 1.27 1.27)) hide)
     )
@@
     )
     (pin "1")
-  )
-  (symbol (lib_id "Mechanical:MountingHole") (at 199.39 81.28 0) (unit 1)
-    (in_bom yes) (on_board yes) (fields_autoplaced)
-    (property "Reference" "H1" (id 0) (at 201.93 80.4453 0)
-      (effects (font (size 1.27 1.27)) (justify left))
-    )
-    (property "Value" "MountingHole" (id 1) (at 201.93 82.9822 0)
-      (effects (font (size 1.27 1.27)) (justify left) hide)
-    )
-    (property "Footprint" "cycfi_library:hole_3mm" (id 2) (at 199.39 81.28 0)
-      (effects (font (size 1.27 1.27)) hide)
-    )
-    (property "Datasheet" "~" (id 3) (at 199.39 81.28 0)
-      (effects (font (size 1.27 1.27)) hide)
-    )
   )
   (symbol (lib_id "Connector_Generic:Conn_02x02_Counter_Clockwise") (at 140.97 71.12 0) (unit 1)
@@
     (pin "4")
   )
-  (symbol (lib_id "Mechanical:MountingHole") (at 199.39 87.63 0) (unit 1)
-    (in_bom yes) (on_board yes) (fields_autoplaced)
-    (property "Reference" "H2" (id 0) (at 201.93 88.0638 0)
-      (effects (font (size 1.27 1.27)) (justify left))
-    )
-    (property "Value" "MountingHole" (id 1) (at 201.93 89.3322 0)
-      (effects (font (size 1.27 1.27)) (justify left) hide)
-    )
-    (property "Footprint" "cycfi_library:hole_3mm" (id 2) (at 199.39 87.63 0)
-      (effects (font (size 1.27 1.27)) hide)
-    )
-    (property "Datasheet" "~" (id 3) (at 199.39 87.63 0)
-      (effects (font (size 1.27 1.27)) hide)
-    )
-  )
   (sheet_instances
     (path "/" (page "1"))
@@
       (reference "#PWR01") (unit 1) (value "GND") (footprint "")
     )
-    (path "/00000000-0000-0000-0000-00006112c732"
-      (reference "#PWR03") (unit 1) (value "GND") (footprint "")
-    )
-    (path "/6f1beb86-67e1-46bf-8c2b-6d1e1485d5c0"
-      (reference "H1") (unit 1) (value "MountingHole") (footprint "cycfi_library:hole_3mm")
-    )
-    (path "/b90f2dfd-9639-4bac-9825-9f33089900c6"
-      (reference "H2") (unit 1) (value "MountingHole") (footprint "cycfi_library:hole_3mm")
-    )
-    (path "/00000000-0000-0000-0000-00006112bc09"
-      (reference "H5") (unit 1) (value "single_pad") (footprint "xr_spectra_library:rail_slot_3.5")
-    )
-    (path "/00000000-0000-0000-0000-00006114c19e"
-      (reference "H6") (unit 1) (value "single_pad") (footprint "xr_spectra_library:rail_slot_3.5")
-    )
     (path "/00000000-0000-0000-0000-000061122909"
-      (reference "IC1") (unit 1) (value "single_pad") (footprint "cycfi_library:single-pad-1.6x1.6_circular")
+      (reference "IC1") (unit 1) (value "single_pad") (footprint "Connector_PinHeader_2.54mm:PinHeader_1x01_P2.54mm_Vertical")
     )
     (path "/00000000-0000-0000-0000-00006112ffae"
-      (reference "IC2") (unit 1) (value "single_pad") (footprint "cycfi_library:single-pad-1.6x1.6_circular")
+      (reference "IC2") (unit 1) (value "single_pad") (footprint "Connector_PinHeader_2.54mm:PinHeader_1x01_P2.54mm_Vertical")
     )
     (path "/8d2043d0-1e2a-47a8-b40c-1d3c6b8242cf"
@@
     )
     (path "/00000000-0000-0000-0000-000061122fed"
-      (reference "OC1") (unit 1) (value "single_pad") (footprint "cycfi_library:single-pad-1.6x1.6_circular")
+      (reference "OC1") (unit 1) (value "single_pad") (footprint "Connector_PinHeader_2.54mm:PinHeader_1x01_P2.54mm_Vertical")
     )
     (path "/00000000-0000-0000-0000-0000611302a2"
-      (reference "OC2") (unit 1) (value "single_pad") (footprint "cycfi_library:single-pad-1.6x1.6_circular")
-    )
-  )
+      (reference "OC2") (unit 1) (value "single_pad") (footprint "Connector_PinHeader_2.54mm:PinHeader_1x01_P2.54mm_Vertical")
+    )
+  )
