File: hardware/output_board/output_board.kicad_sch (KiCad schematic)
At the start: 6 parts, among them J1 I/O, J2 conn_2x2

Commit message: Rename and minor refinements
Parts:
- removed H1, H2, H3, H4: MountingHole, cycfi_library:mounting_hole_st1.9, symbol Mechanical:MountingHole
Connections:
- net middle_coil: now reaches J2.1 (Pin_1)
- no-connect marks 1 -> 0
Other:
- title: XR Spectra Passive Board -> XR Spectra Output Board
Changed lines of the file:
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@@
   (paper "A4")
   (title_block
-    (title "XR Spectra Passive Board")
-    (date "2024-11-30")
+    (title "XR Spectra Output Board")
+    (date "2024-12-01")
     (rev "3.0")
     (company "Document No. 2022013")
@@
   (junction (at 110.49 74.93) (diameter 0) (color 0 0 0 0)
   )
-  (no_connect (at 109.22 111.76))
   (wire (pts (xy 106.68 58.42) (xy 113.03 58.42))
     (stroke (width 0) (type default) (color 0 0 0 0))
@@
     )
   )
+  (global_label "middle_coil" (shape input) (at 109.22 111.76 180) (fields_autoplaced)
+    (effects (font (size 1.27 1.27)) (justify right))
+    (property "Intersheet References" "${INTERSHEET_REFS}" (id 0) (at 96.0706 111.6806 0)
+      (effects (font (size 1.27 1.27)) (justify right) hide)
+    )
+  )
   (global_label "out-" (shape input) (at 121.92 114.3 0) (fields_autoplaced)
     (effects (font (size 1.27 1.27)) (justify left))
@@
     (effects (font (size 1.27 1.27)) (justify left))
     (property "Intersheet References" "${INTERSHEET_REFS}" (id 0) (at -5.08 1.27 0)
-      (effects (font (size 1.27 1.27)) hide)
-    )
-  )
-  (symbol (lib_id "Mechanical:MountingHole") (at 217.17 55.88 0) (unit 1)
-    (in_bom yes) (on_board yes)
-    (property "Reference" "H1" (id 0) (at 219.71 54.7116 0)
-      (effects (font (size 1.27 1.27)) (justify left))
-    )
-    (property "Value" "MountingHole" (id 1) (at 219.71 57.023 0)
-      (effects (font (size 1.27 1.27)) (justify left))
-    )
-    (property "Footprint" "cycfi_library:mounting_hole_st1.9" (id 2) (at 217.17 55.88 0)
-      (effects (font (size 1.27 1.27)) hide)
-    )
-    (property "Datasheet" "~" (id 3) (at 217.17 55.88 0)
-      (effects (font (size 1.27 1.27)) hide)
-    )
-  )
-  (symbol (lib_id "Mechanical:MountingHole") (at 217.17 60.96 0) (unit 1)
-    (in_bom yes) (on_board yes)
-    (property "Reference" "H2" (id 0) (at 219.71 59.7916 0)
-      (effects (font (size 1.27 1.27)) (justify left))
-    )
-    (property "Value" "MountingHole" (id 1) (at 219.71 62.103 0)
-      (effects (font (size 1.27 1.27)) (justify left))
-    )
-    (property "Footprint" "cycfi_library:mounting_hole_st1.9" (id 2) (at 217.17 60.96 0)
-      (effects (font (size 1.27 1.27)) hide)
-    )
-    (property "Datasheet" "~" (id 3) (at 217.17 60.96 0)
-      (effects (font (size 1.27 1.27)) hide)
-    )
-  )
-  (symbol (lib_id "Mechanical:MountingHole") (at 217.17 66.04 0) (unit 1)
-    (in_bom yes) (on_board yes)
-    (property "Reference" "H3" (id 0) (at 219.71 64.8716 0)
-      (effects (font (size 1.27 1.27)) (justify left))
-    )
-    (property "Value" "MountingHole" (id 1) (at 219.71 67.183 0)
-      (effects (font (size 1.27 1.27)) (justify left))
-    )
-    (property "Footprint" "cycfi_library:mounting_hole_st1.9" (id 2) (at 217.17 66.04 0)
-      (effects (font (size 1.27 1.27)) hide)
-    )
-    (property "Datasheet" "~" (id 3) (at 217.17 66.04 0)
-      (effects (font (size 1.27 1.27)) hide)
-    )
-  )
-  (symbol (lib_id "Mechanical:MountingHole") (at 217.17 71.12 0) (unit 1)
-    (in_bom yes) (on_board yes)
-    (property "Reference" "H4" (id 0) (at 219.71 69.9516 0)
-      (effects (font (size 1.27 1.27)) (justify left))
-    )
-    (property "Value" "MountingHole" (id 1) (at 219.71 72.263 0)
-      (effects (font (size 1.27 1.27)) (justify left))
-    )
-    (property "Footprint" "cycfi_library:mounting_hole_st1.9" (id 2) (at 217.17 71.12 0)
-      (effects (font (size 1.27 1.27)) hide)
-    )
-    (property "Datasheet" "~" (id 3) (at 217.17 71.12 0)
       (effects (font (size 1.27 1.27)) hide)
     )
@@
   (symbol (lib_id "power:GND") (at 144.78 66.04 0) (unit 1)
     (in_bom yes) (on_board yes)
-    (property "Reference" "#PWR?" (id 0) (at 144.78 72.39 0)
+    (property "Reference" "#PWR0101" (id 0) (at 144.78 72.39 0)
       (effects (font (size 1.27 1.27)) hide)
     )
@@
     )
     (path "/733121c4-8a56-41fb-ad2d-f02f2cc58dc5"
-      (reference "#PWR?") (unit 1) (value "GND") (footprint "")
-    )
-    (path "/00000000-0000-0000-0000-000060cc8e41"
-      (reference "H1") (unit 1) (value "MountingHole") (footprint "cycfi_library:mounting_hole_st1.9")
-    )
-    (path "/00000000-0000-0000-0000-000060cc94f0"
-      (reference "H2") (unit 1) (value "MountingHole") (footprint "cycfi_library:mounting_hole_st1.9")
-    )
-    (path "/00000000-0000-0000-0000-000060cca720"
-      (reference "H3") (unit 1) (value "MountingHole") (footprint "cycfi_library:mounting_hole_st1.9")
-    )
-    (path "/00000000-0000-0000-0000-000060ccabb9"
-      (reference "H4") (unit 1) (value "MountingHole") (footprint "cycfi_library:mounting_hole_st1.9")
+      (reference "#PWR0101") (unit 1) (value "GND") (footprint "")
     )
     (path "/00000000-0000-0000-0000-000060fa7e20"
