File: hardware/output_board/output_board.kicad_pcb (KiCad board)
At the start: 2 copper layers, 45 x 17 mm, 7 parts, among them J1 I/O, J2 conn_2x2

Commit message: Rename and minor refinements
Connections:
- J2 pad 1: unconnected-(J2-Pad1) -> middle_coil
Other:
- board text added: "IC1"
- board text added: "IC2"
- board text added: "OC1/2"
- board text removed: "INT_COIL+"
- board text removed: "OUT-"
- board text removed: "X"
Changed lines of the file:
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@@
   (net 4 "int_coil+")
   (net 5 "out-")
-  (net 6 "unconnected-(J2-Pad1)")
+  (net 6 "middle_coil")
   (footprint "cycfi_library:mounting_hole_st1.9" (layer "F.Cu")
     (at 148 115 180)
@@
     (property "Sheetfile" "passive.kicad_sch")
     (property "Sheetname" "")
-    (attr exclude_from_pos_files)
+    (attr board_only exclude_from_pos_files)
     (fp_text reference "H1" (at 0 -3.2) (layer "F.SilkS") hide
       (effects (font (size 1 1) (thickness 0.15)))
@@
     (property "Sheetfile" "passive.kicad_sch")
     (property "Sheetname" "")
-    (attr exclude_from_pos_files)
+    (attr board_only exclude_from_pos_files)
     (fp_text reference "H2" (at 0 -3.2) (layer "F.SilkS") hide
       (effects (font (size 1 1) (thickness 0.15)))
@@
     (property "Sheetfile" "passive.kicad_sch")
     (property "Sheetname" "")
-    (attr exclude_from_pos_files)
+    (attr board_only exclude_from_pos_files)
     (fp_text reference "H3" (at 0 -3.2) (layer "F.SilkS") hide
       (effects (font (size 1 1) (thickness 0.15)))
@@
     (property "Sheetfile" "passive.kicad_sch")
     (property "Sheetname" "")
-    (attr exclude_from_pos_files)
+    (attr board_only exclude_from_pos_files)
     (fp_text reference "H4" (at 0 -3.2) (layer "F.SilkS") hide
       (effects (font (size 1 1) (thickness 0.15)))
@@
     (descr "surface-mounted straight pin socket, 2x2, 2.00mm pitch, double rows")
     (tags "Surface mounted pin header SMD 2x2 200mm double row")
-    (property "Sheetfile" "passive.kicad_sch")
+    (property "Sheetfile" "File: output_board.kicad_sch")
     (property "Sheetname" "")
     (attr smd)
@@
     (pad "" np_thru_hole circle (at 0 0) (size 1.1 1.1) (drill 1.02) (layers F&B.Cu *.Mask))
     (pad "1" smd rect (at -2.275 -1) (size 2.65 0.8) (layers "F.Cu" "F.Paste" "F.Mask")
-      (net 6 "unconnected-(J2-Pad1)") (pinfunction "Pin_1") (pintype "passive+no_connect"))
+      (net 6 "middle_coil") (pinfunction "Pin_1") (pintype "passive"))
     (pad "2" smd rect (at -2.275 1) (size 2.65 0.8) (layers "F.Cu" "F.Paste" "F.Mask")
       (net 1 "GND") (pinfunction "Pin_2") (pintype "passive"))
@@
   (footprint "cycfi_library:pin_header_2x5p_2.54mm_smd_horizontal" (layer "B.Cu")
     (at 118.9 108.58)
-    (property "Sheetfile" "passive.kicad_sch")
+    (property "Sheetfile" "File: output_board.kicad_sch")
     (property "Sheetname" "")
     (attr through_hole)
@@
     (effects (font (size 0.5 0.5) (thickness 0.125)) (justify mirror))
   )
-  (gr_text "X" (at 133.5 107.45) (layer "F.SilkS")
+  (gr_text "OC1/2" (at 132 107.4) (layer "F.SilkS")
     (effects (font (size 0.8 0.8) (thickness 0.1)))
   )
-  (gr_text "OUT-" (at 143.85 109.45) (layer "F.SilkS")
+  (gr_text "IC2" (at 143.25 109.5) (layer "F.SilkS")
     (effects (font (size 0.8 0.8) (thickness 0.1)))
   )
-  (gr_text "INT_COIL+" (at 145.25 107.55) (layer "F.SilkS")
+  (gr_text "IC1" (at 143.25 107.55) (layer "F.SilkS")
     (effects (font (size 0.8 0.8) (thickness 0.1)))
   )
-  (gr_text "GND" (at 132.55 109.5) (layer "F.SilkS")
+  (gr_text "GND" (at 132.75 109.5) (layer "F.SilkS")
     (effects (font (size 0.8 0.8) (thickness 0.1)))
   )
   (via (at 136.6 113.2) (size 0.8) (drill 0.4) (layers "F.Cu" "B.Cu") (free) (net 1))
   (via (at 135.1 113.2) (size 0.8) (drill 0.4) (layers "F.Cu" "B.Cu") (free) (net 1))
-  (via (at 113.5 104.5) (size 0.8) (drill 0.4) (layers "F.Cu" "B.Cu") (free) (net 1))
-  (via (at 112 104.5) (size 0.8) (drill 0.4) (layers "F.Cu" "B.Cu") (free) (net 1))
-  (via (at 113.5 106) (size 0.8) (drill 0.4) (layers "F.Cu" "B.Cu") (free) (net 1))
+  (via (at 116.5 104.75) (size 0.8) (drill 0.4) (layers "F.Cu" "B.Cu") (free) (net 1))
+  (via (at 116.5 107.25) (size 0.8) (drill 0.4) (layers "F.Cu" "B.Cu") (free) (net 1))
+  (via (at 121.25 104.75) (size 0.8) (drill 0.4) (layers "F.Cu" "B.Cu") (free) (net 1))
   (via (at 136.6 111.7) (size 0.8) (drill 0.4) (layers "F.Cu" "B.Cu") (free) (net 1))
   (via (at 135.1 111.7) (size 0.8) (drill 0.4) (layers "F.Cu" "B.Cu") (free) (net 1))
-  (via (at 112 106) (size 0.8) (drill 0.4) (layers "F.Cu" "B.Cu") (free) (net 1))
+  (via (at 121.25 107.25) (size 0.8) (drill 0.4) (layers "F.Cu" "B.Cu") (free) (net 1))
   (segment (start 121.3044 103.5) (end 123.5 103.5) (width 0.2) (layer "B.Cu") (net 2))
   (segment (start 123.34 113.66) (end 121.3044 113.66) (width 0.2) (layer "B.Cu") (net 2))

Commit message: Final refinements
Parts:
- removed the G*** at (145.2, 108.5)
- added G***: LOGO, cycfi_library:cycfi-logo-9mm, B.Cu at (146.4, 109.0)
- moved H3 5.52 mm to (112.5, 115.5)
- moved H4 5.52 mm to (112.5, 102.5)
- moved J2 3.04 mm to (141.0, 109.0)
- moved H1 0.71 mm to (147.5, 115.5)
- moved H2 0.71 mm to (147.5, 102.5)
- moved J1 0.50 mm to (118.9, 109.1)
Routing:
- net out-: track 36.6 -> 39.9 mm
- net int_coil+: track 31.3 -> 33.4 mm
Other:
- board size 45 x 17 mm -> 40 x 18 mm

Commit message: Change name
Other:
- board text added: "XR Spectra v3.0"
- board text removed: "XR Spectra Passive v3.0"
Changed lines of the file:
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@@
 		(layer "Edge.Cuts")
 	)
-	(gr_text "XR Spectra \nPassive v3.0"
-		(at 147.985786 109.285786 90)
+	(gr_text "XR Spectra v3.0"
+		(at 147.585786 109.285786 90)
 		(layer "B.SilkS")
 		(effects
