File: hardware/base_board/base_board_60/base_board_60.kicad_sch (KiCad schematic)
At the start: 5 parts, among them IC1 single_pad, IC2 single_pad, J1 conn_2x2

Commit message: Moved coil solder pads to outer perimeter
Parts:
- IC1, IC2, OC1, OC2: footprint Connector_PinHeader_2.54mm:PinHeader_1x01_P2.54mm_Vertical -> cycfi_library:xr_spectra_coil_pads
Changed lines of the file:
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@@
 			)
 		)
-		(property "Footprint" "Connector_PinHeader_2.54mm:PinHeader_1x01_P2.54mm_Vertical"
+		(property "Footprint" "cycfi_library:xr_spectra_coil_pads"
 			(at 172.72 71.12 0)
 			(effects
@@
 			)
 		)
-		(property "Footprint" "Connector_PinHeader_2.54mm:PinHeader_1x01_P2.54mm_Vertical"
+		(property "Footprint" "cycfi_library:xr_spectra_coil_pads"
 			(at 172.72 77.47 0)
 			(effects
@@
 			)
 		)
-		(property "Footprint" "Connector_PinHeader_2.54mm:PinHeader_1x01_P2.54mm_Vertical"
+		(property "Footprint" "cycfi_library:xr_spectra_coil_pads"
 			(at 172.72 90.17 0)
 			(effects
@@
 			)
 		)
-		(property "Footprint" "Connector_PinHeader_2.54mm:PinHeader_1x01_P2.54mm_Vertical"
+		(property "Footprint" "cycfi_library:xr_spectra_coil_pads"
 			(at 172.72 83.82 0)
 			(effects

Commit message: Reversing the coil polarity
Parts:
- renumbered OC1 to IC1, OC2 to IC2, IC1 to OC1, IC2 to OC2
Changed lines of the file:
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@@
 		(on_board yes)
 		(dnp no)
-		(property "Reference" "IC1"
+		(property "Reference" "OC1"
 			(at 175.895 71.12 90)
 			(effects
@@
 			(project ""
 				(path "/b994142f-02ac-4881-9587-6d3df53c96d2"
-					(reference "IC1")
+					(reference "OC1")
 					(unit 1)
 				)
@@
 		(on_board yes)
 		(dnp no)
-		(property "Reference" "OC1"
+		(property "Reference" "IC1"
 			(at 175.895 77.47 90)
 			(effects
@@
 			(project ""
 				(path "/b994142f-02ac-4881-9587-6d3df53c96d2"
-					(reference "OC1")
+					(reference "IC1")
 					(unit 1)
 				)
@@
 		(on_board yes)
 		(dnp no)
-		(property "Reference" "IC2"
+		(property "Reference" "OC2"
 			(at 175.895 90.17 90)
 			(effects
@@
 			(project ""
 				(path "/b994142f-02ac-4881-9587-6d3df53c96d2"
-					(reference "IC2")
+					(reference "OC2")
 					(unit 1)
 				)
@@
 		(on_board yes)
 		(dnp no)
-		(property "Reference" "OC2"
+		(property "Reference" "IC2"
 			(at 175.895 83.82 90)
 			(effects
@@
 			(project ""
 				(path "/b994142f-02ac-4881-9587-6d3df53c96d2"
-					(reference "OC2")
-					(unit 1)
-				)
+					(reference "IC2")
+					(unit 1)
+				)
